File: anthropic-macropad.kicad_pcb (KiCad board)
At the start: 2 copper layers, 136 x 81 mm, 12 parts, among them SW1 ESC, SW10 ENTER, SW11 MIC, SW2 TAB, SW3 ALLOW_ONCE, SW4 UP, SW5 ALLOW_ALWAYS, SW6 LEFT, SW7 DOWN, SW8 RIGHT, SW9 REJECT, U1 XIAO_RP2040

Commit message: Route PCB and reshape board outline
- Autorouted all traces via Freerouting (F.Cu + B.Cu)
- Reshaped head to flat wide top matching space invader reference
- Moved XIAO RP2040 to front with exposed USB-C at top edge
- Moved ESC/TAB to eye positions in the head
- Removed legs (case will provide them)
- Spaced bottom row keys for 2u ENTER clearance
- DRC clean: 0 errors, 0 unconnected pads

Co-Authored-By: Claude Opus 4.6 <noreply@anthropic.com>
Routing:
- net GND: track 0.00 -> 299.2 mm
- net SW_REJECT: track 0.00 -> 88.2 mm, vias 0 -> 1
- net SW_ALLOW_ALWAYS: track 0.00 -> 76.6 mm
- net SW_MIC: track 0.00 -> 70.9 mm
- net SW_ALLOW_ONCE: track 0.00 -> 66.2 mm, vias 0 -> 1
- net SW_ENTER: track 0.00 -> 60.5 mm
- net SW_RIGHT: track 0.00 -> 39.7 mm
- net SW_TAB: track 0.00 -> 36.8 mm
- net SW_LEFT: track 0.00 -> 32.5 mm
- net SW_DOWN: track 0.00 -> 30.8 mm
- net SW_UP: track 0.00 -> 19.1 mm
- net SW_ESC: track 0.00 -> 17.5 mm

Commit message: Add GND copper pour on B.Cu and remove redundant GND traces
Replaced 30 individual GND trace segments with a B.Cu ground
pour that covers the entire board area.

Co-Authored-By: Claude Opus 4.6 <noreply@anthropic.com>
Routing:
- net GND: track 299.2 -> 0.00 mm
- added copper zone on B.Cu, net GND
Changed lines of the file:
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@@
-	)
-	(segment
-		(start 96.19 76.432)
-		(end 96.19 76.46)
-		(width 0.2)
-		(layer "F.Cu")
-		(net "GND")
-	)
-	(segment
-		(start 39.1232 66.3932)
-		(end 39.1232 68.7843)
-		(width 0.2)
-		(layer "F.Cu")
-		(net "GND")
-	)
-	(segment
-		(start 154.19 65.46)
-		(end 126.19 65.46)
-		(width 0.2)
-		(layer "F.Cu")
-		(net "GND")
-	)
-	(segment
-		(start 38.19 65.46)
-		(end 39.1232 66.3932)
-		(width 0.2)
-		(layer "F.Cu")
-		(net "GND")
-	)
-	(segment
-		(start 121.19 41.46)
-		(end 111.24 41.46)
-		(width 0.2)
-		(layer "F.Cu")
-		(net "GND")
-	)
-	(segment
-		(start 111.24 41.46)
-		(end 107.62 45.08)
-		(width 0.2)
-		(layer "F.Cu")
-		(net "GND")
-	)
-	(segment
-		(start 96.19 76.432)
-		(end 77.218 76.432)
-		(width 0.2)
-		(layer "F.Cu")
-		(net "GND")
-	)
-	(segment
-		(start 115.162 76.432)
-		(end 96.19 76.432)
-		(width 0.2)
-		(layer "F.Cu")
-		(net "GND")
-	)
-	(segment
-		(start 126.19 65.46)
-		(end 115.19 76.46)
-		(width 0.2)
-		(layer "F.Cu")
-		(net "GND")
-	)
-	(segment
-		(start 77.218 76.432)
-		(end 77.19 76.46)
-		(width 0.2)
-		(layer "F.Cu")
-		(net "GND")
-	)
-	(segment
-		(start 46.7989 76.46)
-		(end 77.19 76.46)
-		(width 0.2)
-		(layer "F.Cu")
-		(net "GND")
-	)
-	(segment
-		(start 39.1232 68.7843)
-		(end 46.7989 76.46)
-		(width 0.2)
-		(layer "F.Cu")
-		(net "GND")
-	)
-	(segment
-		(start 115.19 76.46)
-		(end 115.162 76.432)
-		(width 0.2)
-		(layer "F.Cu")
-		(net "GND")
-	)
-	(segment
-		(start 115.19 76.46)
-		(end 115.19 52.65)
-		(width 0.2)
-		(layer "B.Cu")
-		(net "GND")
-	)
-	(segment
-		(start 76.3794 76.46)
-		(end 77.19 76.46)
-		(width 0.2)
-		(layer "B.Cu")
-		(net "GND")
-	)
-	(segment
-		(start 66.19 86.6494)
-		(end 76.3794 76.46)
-		(width 0.2)
-		(layer "B.Cu")
-		(net "GND")
-	)
-	(segment
-		(start 71.3902 41.6602)
-		(end 71.3902 71.4708)
-		(width 0.2)
-		(layer "B.Cu")
-		(net "GND")
-	)
-	(segment
-		(start 66.19 95.46)
-		(end 66.19 86.6494)
-		(width 0.2)
-		(layer "B.Cu")
-		(net "GND")
-	)
-	(segment
-		(start 115.4273 76.6973)
-		(end 115.19 76.46)
-		(width 0.2)
-		(layer "B.Cu")
-		(net "GND")
-	)
-	(segment
-		(start 96.3679 95.2821)
-		(end 96.3679 76.6379)
-		(width 0.2)
-		(layer "B.Cu")
-		(net "GND")
-	)
-	(segment
-		(start 96.3679 76.6379)
-		(end 96.19 76.46)
-		(width 0.2)
-		(layer "B.Cu")
-		(net "GND")
-	)
-	(segment
-		(start 126.19 95.46)
-		(end 115.4273 84.6973)
-		(width 0.2)
-		(layer "B.Cu")
-		(net "GND")
-	)
-	(segment
-		(start 96.19 95.46)
-		(end 96.3679 95.2821)
-		(width 0.2)
-		(layer "B.Cu")
-		(net "GND")
-	)
-	(segment
-		(start 96.19 57.46)
-		(end 96.3467 57.6167)
-		(width 0.2)
-		(layer "B.Cu")
-		(net "GND")
-	)
-	(segment
-		(start 115.4273 84.6973)
-		(end 115.4273 76.6973)
-		(width 0.2)
-		(layer "B.Cu")
-		(net "GND")
-	)
-	(segment
-		(start 71.19 41.46)
-		(end 71.3902 41.6602)
-		(width 0.2)
-		(layer "B.Cu")
-		(net "GND")
-	)
-	(segment
-		(start 96.3467 57.6167)
-		(end 96.3467 76.3033)
-		(width 0.2)
-		(layer "B.Cu")
-		(net "GND")
-	)
-	(segment
-		(start 115.19 52.65)
-		(end 107.62 45.08)
-		(width 0.2)
-		(layer "B.Cu")
-		(net "GND")
-	)
-	(segment
-		(start 96.3467 76.3033)
-		(end 96.19 76.46)
-		(width 0.2)
-		(layer "B.Cu")
-		(net "GND")
-	)
-	(segment
-		(start 71.3902 71.4708)
-		(end 76.3794 76.46)
-		(width 0.2)
-		(layer "B.Cu")
-		(net "GND")
 	)
 	(segment
@@
 		(net "SW_MIC")
 	)
+	(zone
+		(net "GND")
+		(layer "B.Cu")
+		(hatch edge 0.5)
+		(connect_pads
+			(clearance 0.3)
+		)
+		(min_thickness 0.2)
+		(fill yes
+			(thermal_gap 0.5)
+			(thermal_bridge_width 0.5)
+		)
+		(polygon
+			(pts
+				(xy 30 20) (xy 170 20) (xy 170 115) (xy 30 115)
+			)
+		)
+	)
 	(embedded_fonts no)
