File: claude-macropad-more-track-width.kicad_pcb (KiCad board)
At the start: 2 copper layers, 136 x 81 mm, 16 parts, among them SW1 ESC, SW10 ENTER, SW11 MIC, SW2 TAB, SW3 ALLOW_ONCE, SW4 UP, SW5 ALLOW_ALWAYS, SW6 LEFT, SW7 DOWN, SW8 RIGHT, SW9 REJECT, U1 XIAO_RP2040

Commit message: Rename project from anthropic-macropad to claude-macropad
Co-Authored-By: Claude Opus 4.6 <noreply@anthropic.com>
Routing:
- net SW_ALLOW_ALWAYS: track 76.6 -> 91.7 mm
Changed lines of the file:
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@@
 	)
 	(segment
-		(start 113.1649 62.92)
+		(start 92.38 42.54)
+		(end 88 46.92)
+		(width 0.3)
+		(layer "F.Cu")
+		(net "SW_ALLOW_ALWAYS")
+	)
+	(segment
+		(start 94.08 62.92)
 		(end 160.54 62.92)
 		(width 0.3)
@@
 	)
 	(segment
-		(start 92.7849 42.54)
-		(end 113.1649 62.92)
+		(start 94 63)
+		(end 94.08 62.92)
 		(width 0.3)
 		(layer "F.Cu")
+		(net "SW_ALLOW_ALWAYS")
+	)
+	(segment
+		(start 88 57)
+		(end 94 63)
+		(width 0.3)
+		(layer "F.Cu")
+		(net "SW_ALLOW_ALWAYS")
+	)
+	(segment
+		(start 88 46.92)
+		(end 88 57)
+		(width 0.3)
+		(layer "F.Cu")
